File: Hardware/Block_Template.sch (EAGLE design)
At the start: 9 parts, among them U2 EDISON_CONNECTOR_FULLMOUNTING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, U3 EDISON_CONNECTOR_FULLHEADER

Commit message: updated footprints to remove jumpers between connector pins. Renamed Connectors to J1 and J2. Locked vias, holes, connectors, and logos.  Trying to keep things standard for future builds
Parts:
- renumbered U2 to J1, U3 to J2
